File: PCCode/disposable_heroes/Kicad_relesSR/VISIR_Lei_Ohm/VISIR_Lei_Ohm.kicad_sch (KiCad schematic)
At the start: 23 parts, among them J1 Raspberry PI5, J2 Fonte dc, J3 Fonte 12V, J4 Fonte 5V, K1 3572-1220-123, K2 3572-1220-123, K3 3572-1220-123, K4 3570-1331-123, K5 3570-1331-123, K6 3572-1220-123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

Commit message: update schematic KICAD
Connections:
- net A: no longer MES1.2 (+)
- net D: no longer K5.4
- new net: K5.4, MES1.2 (+)
Other:
- note added: "VER LIGAÇÃO DO AMPERÍMETRO 1 liga ao 7"
- moved on the sheet: MES1
Changed lines of the file:
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@@
 (kicad_sch (version 20230121) (generator eeschema)
   (paper "A3")
-  (junction (at 42.7736 109.728) (diameter 0) (color 0 0 0 0)
-  )
   (junction (at 83.058 113.919) (diameter 0) (color 0 0 0 0)
   )
@@
   )
   (junction (at 157.7848 94.488) (diameter 0) (color 0 0 0 0)
-  )
-  (junction (at 22.352 109.728) (diameter 0) (color 0 0 0 0)
   )
   (junction (at 71.12 131.572) (diameter 0) (color 0 0 0 0)
@@
     (stroke (width 0) (type default) (color 0 0 0 1))
   )
-  (wire (pts (xy 20.1168 109.7788) (xy 22.352 109.7788))
-    (stroke (width 0) (type default) (color 255 0 0 1))
-  )
   (wire (pts (xy 58.42 131.572) (xy 71.12 131.572))
     (stroke (width 0) (type default))
@@
     (stroke (width 0) (type default))
   )
+  (wire (pts (xy 22.352 105.664) (xy 22.352 109.728))
+    (stroke (width 0) (type default) (color 255 0 0 1))
+  )
   (wire (pts (xy 46.355 59.309) (xy 39.37 59.309))
     (stroke (width 0) (type default))
@@
     (stroke (width 0) (type default) (color 255 255 0 1))
   )
+  (wire (pts (xy 37.0332 122.6312) (xy 42.7736 122.6312))
+    (stroke (width 0) (type default))
+  )
   (wire (pts (xy 200.4822 44.0944) (xy 211.2772 44.0944))
     (stroke (width 0) (type default))
@@
   (wire (pts (xy 231.267 115.951) (xy 235.204 115.951))
     (stroke (width 0) (type default) (color 255 255 0 1))
+  )
+  (wire (pts (xy 42.7736 109.728) (xy 42.7736 112.4712))
+    (stroke (width 0) (type default) (color 0 0 0 1))
   )
   (wire (pts (xy 231.267 80.391) (xy 235.204 80.391))
@@
     (stroke (width 0) (type default))
   )
-  (wire (pts (xy 42.7736 106.2228) (xy 42.7736 109.728))
-    (stroke (width 0) (type default) (color 0 0 0 1))
-  )
   (wire (pts (xy 80.01 113.919) (xy 83.058 113.919))
     (stroke (width 0) (type default))
@@
     (stroke (width 0) (type default))
   )
-  (wire (pts (xy 22.352 109.7788) (xy 22.352 109.728))
-    (stroke (width 0) (type default) (color 255 0 0 1))
-  )
   (wire (pts (xy 22.1488 171.6024) (xy 22.1488 174.0154))
     (stroke (width 0) (type default))
+  )
+  (wire (pts (xy 38.862 109.728) (xy 42.7736 109.728))
+    (stroke (width 0) (type default) (color 0 0 0 1))
   )
   (wire (pts (xy 161.417 59.3344) (xy 164.9222 59.3344))
@@
     (stroke (width 0) (type default))
   )
-  (wire (pts (xy 18.8214 110.7186) (xy 20.1168 109.7788))
-    (stroke (width 0) (type default) (color 255 0 0 1))
-  )
   (wire (pts (xy 121.92 24.765) (xy 121.92 27.686))
     (stroke (width 0) (type default))
@@
   (wire (pts (xy 42.926 51.3842) (xy 46.3296 51.3842))
     (stroke (width 0) (type default))
-  )
-  (wire (pts (xy 42.7736 124.9426) (xy 42.7736 109.728))
-    (stroke (width 0) (type default) (color 0 0 0 1))
   )
   (wire (pts (xy 231.267 105.791) (xy 235.204 105.791))
@@
     (stroke (width 0) (type default))
   )
-  (wire (pts (xy 22.352 106.1466) (xy 22.352 109.728))
-    (stroke (width 0) (type default) (color 255 0 0 1))
-  )
   (wire (pts (xy 82.7532 181.0512) (xy 51.181 181.0512))
     (stroke (width 0.254) (type dash) (color 132 0 0 1))
@@
     (stroke (width 0) (type default))
   )
-  (wire (pts (xy 18.8214 110.7186) (xy 18.8214 113.411))
-    (stroke (width 0) (type default) (color 255 0 0 1))
-  )
-  (wire (pts (xy 38.862 109.728) (xy 42.7736 109.728))
-    (stroke (width 0) (type default) (color 0 0 0 1))
-  )
   (wire (pts (xy 66.802 28.829) (xy 67.945 27.686))
     (stroke (width 0) (type default))
@@
     (stroke (width 0.254) (type dash) (color 0 0 255 1))
   )
-  (wire (pts (xy 18.8214 124.9426) (xy 42.7736 124.9426))
-    (stroke (width 0) (type default) (color 0 0 0 1))
-  )
   (wire (pts (xy 115.697 61.976) (xy 122.047 61.976))
     (stroke (width 0) (type default))
@@
     (stroke (width 0.254) (type dash) (color 132 0 0 1))
   )
-  (wire (pts (xy 18.8214 124.9426) (xy 18.8214 123.571))
-    (stroke (width 0) (type default) (color 0 0 0 1))
-  )
   (wire (pts (xy 16.6116 105.3084) (xy 16.6116 112.2426))
     (stroke (width 0) (type default))
@@
     (fill (type none))
     (effects (font (size 1.27 1.27)) (justify left top))
+  )
+  (text "VER LIGAÇÃO DO AMPERÍMETRO\n1 liga ao 7" (at 55.0672 128.6764 0)
+    (effects (font (size 1.27 1.27)) (justify left bottom))
   )
   (text "Relé K9 confere mais versatilidade, \njá que pode tornar o ramo do Amperímetro \"independente\""
@@
     )
   )
+  (global_label "D" (shape input) (at 37.0332 122.6312 180) (fields_autoplaced)
+    (effects (font (size 1.27 1.27)) (justify right))
+    (property "Intersheetrefs" "${INTERSHEET_REFS}" (at 32.778 122.6312 0)
+      (effects (font (size 1.27 1.27)) (justify right) hide)
+    )
+  )
   (global_label "B" (shape input) (at 44.3738 131.9784 90) (fields_autoplaced)
     (effects (font (size 1.27 1.27)) (justify left))
@@
     )
   )
-  (global_label "D" (shape input) (at 42.7736 106.2228 90) (fields_autoplaced)
-    (effects (font (size 1.27 1.27)) (justify left))
-    (property "Intersheetrefs" "${INTERSHEET_REFS}" (at 42.7736 101.9676 90)
-      (effects (font (size 1.27 1.27)) (justify left) hide)
-    )
-  )
   (global_label "GND" (shape input) (at 274.193 75.311 0) (fields_autoplaced)
     (effects (font (size 1.27 1.27)) (justify left))
@@
     )
   )
-  (global_label "A" (shape input) (at 22.352 106.1466 90) (fields_autoplaced)
+  (global_label "A" (shape input) (at 22.352 105.664 90) (fields_autoplaced)
     (effects (font (size 1.27 1.27)) (justify left))
-    (property "Intersheetrefs" "${INTERSHEET_REFS}" (at 22.352 102.0728 90)
+    (property "Intersheetrefs" "${INTERSHEET_REFS}" (at 22.352 101.5902 90)
       (effects (font (size 1.27 1.27)) (justify left) hide)
     )
@@
     )
   )
-  (symbol (lib_id "Device:Voltmeter_DC") (at 18.8214 118.491 0) (unit 1)
+  (symbol (lib_id "Device:Voltmeter_DC") (at 42.7736 117.5512 0) (unit 1)
     (in_bom yes) (on_board yes) (dnp no)
-    (property "Reference" "MES1" (at 24.13 119.0752 0)
+    (property "Reference" "MES1" (at 48.0822 118.1354 0)
       (effects (font (size 1.27 1.27)) (justify left))
     )
-    (property "Value" "Voltmeter_DC" (at 23.495 116.0018 0)
+    (property "Value" "Voltmeter_DC" (at 47.4472 115.062 0)
       (effects (font (size 1.27 1.27)) (justify left))
     )
-    (property "Footprint" "Connector_PinHeader_2.54mm:PinHeader_1x02_P2.54mm_Vertical" (at 18.8214 115.951 90)
-      (effects (font (size 1.27 1.27)) hide)
-    )
-    (property "Datasheet" "~" (at 18.8214 115.951 90)
-      (effects (font (size 1.27 1.27)) hide)
-    )
+    (property "Footprint" "Connector_PinHeader_2.54mm:PinHeader_1x02_P2.54mm_Vertical" (at 42.7736 115.0112 90)
+      (effects (font (size 1.27 1.27)) hide)
+    )
+    (property "Datasheet" "~" (at 42.7736 115.0112 90)
+      (effects (font (size 1.27 1.27)) hide)
+    )
